Commit message: adding_arm_robot_model

File: project_arm_1/urdf/project_arm_1.xacro (robot description, xacro)
@@ -1,8 +1,10 @@
-<?xml version="1.0" encoding="utf-8"?>
+<?xml version="1.0"?>
 <!-- This URDF was automatically created by SolidWorks to URDF Exporter! Originally created by Stephen Brawner (brawner@gmail.com)
      Commit Version: 1.6.0-1-g15f4949  Build Version: 1.6.7594.29634
      For more information, please see http://wiki.ros.org/sw_urdf_exporter -->
 <robot
-  name="project_arm_1">
+  name="project_arm_1" xmlns:xacro="http://www.ros.org/wiki/xacro">
+  <!-- Import all Gazebo-customization elements, including Gazebo colors -->
+  <xacro:include filename="$(find project_arm_1)/urdf/project_arm_1.gazebo"/>
    <!-- Used for fixing robot to Gazebo 'base_link' -->
   <link name="world"/>
@@ -269,4 +271,19 @@
     </plugin>
   </gazebo>
+  <gazebo reference="base_robot">
+    <material>Gazebo/Green</material>
+  </gazebo>
+  <gazebo reference="link_1">
+    <material>Gazebo/ZincYellow</material>
+  </gazebo>
+  <gazebo reference="link_2">
+    <material>Gazebo/Red</material>
+  </gazebo>
+  <gazebo reference="link_3">
+    <material>Gazebo/Turquoise</material>
+  </gazebo>
+  <gazebo reference="link_4">
+    <material>Gazebo/Indigo</material>
+  </gazebo>
   <transmission name="trans1">
     <type>transmission_interface/SimpleTransmission</type>
